Commit message: 使用2d激光雷达建图，并且实现amcl定位，还有move_base导航

File: src/unitree_ros/robots/go2_description/xacro/gazebo.xacro (robot description, xacro)
@@ -5,5 +5,4 @@
         <plugin name="gazebo_ros_control" filename="libgazebo_ros_control.so">
             <robotNamespace>go2_gazebo</robotNamespace>
-            <!-- <legacyModeNS>true</legacyModeNS> -->
             <robotSimType>gazebo_ros_control/DefaultRobotHWSim</robotSimType>
         </plugin>
@@ -56,5 +55,5 @@
     </gazebo>
     <!-- Mid360 Livox Gazebo Plugin -->
-    <xacro:property name="M_PI" value="3.14159"/>
+    <!-- <xacro:property name="M_PI" value="3.14159"/>
     <xacro:property name="laser_min_range" value="0.1"/>
     <xacro:property name="laser_max_range" value="200.0"/>
@@ -63,7 +62,7 @@
         <pose>0 0 0 0 0 0</pose>
         <visualize>true</visualize>
-        <update_rate>10</update_rate>
+        <update_rate>10</update_rate> -->
         <!-- 雷达插件，仅用于可视化 -->
-        <plugin name="gazebo_ros_laser_controller" filename="liblivox_laser_simulation.so">
+        <!-- <plugin name="gazebo_ros_laser_controller" filename="liblivox_laser_simulation.so">
         <ray>
             <scan>
@@ -100,7 +99,39 @@
         </plugin>
     </sensor>
+    </gazebo> -->
+    <!-- 2D 激光雷达 -->
+    <gazebo reference="laser_2d">
+    <sensor type="ray" name="laser_2d">
+        <pose>0 0 0 0 0 0</pose>
+        <visualize>true</visualize>
+        <update_rate>10</update_rate>
+        <ray>
+            <scan>
+            <horizontal>
+                <samples>360</samples>
+                <resolution>1</resolution>
+                <min_angle>${-3.14159}</min_angle>
+                <max_angle>${3.14159}</max_angle>
+            </horizontal>
+            </scan>
+            <range>
+            <min>${0.1}</min>
+            <max>30.0</max>
+            <resolution>0.01</resolution>
+            </range>
+            <noise>
+            <type>gaussian</type>
+            <mean>0.0</mean>
+            <stddev>0.01</stddev>
+            </noise>
+        </ray>
+        <plugin name="gazebo_ros_laser_controller" filename="libgazebo_ros_laser.so">
+            <topicName>/scan</topicName>
+            <frameName>laser_2d</frameName>
+        </plugin>
+    </sensor>
     </gazebo>
     <!-- imu -->
-    <gazebo reference="livox_imu_link">
+    <!-- <gazebo reference="livox_imu_link">
         <gravity>true</gravity>
         <sensor name="imu_sensor" type="imu">
@@ -120,5 +151,5 @@
         <pose>0 0 0 0 0 0</pose>
         </sensor>
-    </gazebo>
+    </gazebo> -->
     <!-- Foot contacts. -->
     <gazebo reference="FR_calf">

File: src/unitree_ros/robots/go2_description/xacro/robot.xacro (robot description, xacro)
@@ -89,5 +89,5 @@
     </link>
     <!-- livox mid360 -->
-    <link name="laser_livox">
+    <!-- <link name="laser_livox">
         <collision>
             <origin xyz="0 0 0" rpy="1.57 0 0"/>
@@ -107,6 +107,33 @@
         <parent link="base" />
         <child link="laser_livox"/>
+    </joint> -->
+    <!-- 2D 激光雷达 -->
+    <link name="laser_2d">
+        <visual>
+            <origin xyz="0 0 0" rpy="0 0 0"/>
+            <geometry>
+                <box size="0.05 0.05 0.03"/>
+            </geometry>
+            <material name="red"/>
+        </visual>
+        <collision>
+            <origin xyz="0 0 0" rpy="0 0 0"/>
+            <geometry>
+                <box size="0.05 0.05 0.03"/>
+            </geometry>
+        </collision>
+        <inertial>
+            <mass value="0.05"/>
+            <origin xyz="0 0 0" rpy="0 0 0"/>
+            <inertia ixx="0.0001" ixy="0" ixz="0" iyy="0.0001" iyz="0" izz="0.0001"/>
+        </inertial>
+    </link>
+    <joint name="laser_2d_joint" type="fixed">
+        <origin xyz="0.23 0 0.11" rpy="0 0 0"/>
+        <parent link="base" />
+        <child link="laser_2d"/>
     </joint>
     <!-- imu -->
+    <!--
     <joint name="livox_imu_joint" type="fixed">
         <parent link="laser_livox"/>
@@ -125,5 +152,4 @@
         <box size="0.001 0.001 0.001"/>
         </geometry>
-        <!-- <material name="red"/> -->
         </visual>
         <collision>
@@ -134,4 +160,5 @@
         </collision>
     </link>
+    -->
     <!--
     <joint name="load_joint" type="fixed">
